Commit message: Moveit setup assistant and path exhibition in rviz

File: src/kxsmoveit_robot_description/urdf/arm.xacro (robot description, xacro)
@@ -9,4 +9,10 @@
             <material name="grey"/>
         </visual>
+        <collision>
+            <geometry>
+                <box size="0.4 0.4 0.1"/>
+            </geometry>
+            <origin xyz="0 0 0.05" rpy="0 0 0"/>
+        </collision>
     </link>
     <joint name="joint1" type="revolute">
@@ -25,4 +31,10 @@
             <material name="blue"/>
         </visual>
+        <collision>
+            <geometry>
+                <box size="0.2 0.2 0.5"/>
+            </geometry>
+            <origin xyz="0 0 0.25" rpy="0 0 0"/>
+        </collision>
     </link>
     <joint name="joint2" type="revolute">
@@ -41,4 +53,10 @@
             <material name="grey"/>
         </visual>
+        <collision>
+            <geometry>
+                <cylinder length="0.6" radius="0.05"/>
+            </geometry>
+            <origin xyz="0 0 0.3" rpy="0 0 0"/>
+        </collision>
     </link>
     <joint name="joint3" type="revolute">
@@ -57,4 +75,10 @@
             <material name="blue"/>
         </visual>
+        <collision>
+            <geometry>
+                <cylinder length="0.1" radius="0.05"/>
+            </geometry>
+            <origin xyz="0 0 0.05" rpy="0 0 0"/>
+        </collision>
     </link>
     <joint name="joint4" type="revolute">
@@ -73,4 +97,10 @@
             <material name="grey"/>
         </visual>
+        <collision>
+            <geometry>
+                <cylinder length="0.5" radius="0.05"/>
+            </geometry>
+            <origin xyz="0 0 0.25" rpy="0 0 0"/>
+        </collision>
     </link>
     <joint name="joint5" type="revolute">
@@ -89,4 +119,10 @@
             <material name="blue"/>
         </visual>
+        <collision>
+            <geometry>
+                <box size="0.1 0.1 0.05"/>
+            </geometry>
+            <origin xyz="0 0 0.05" rpy="0 0 0"/>
+        </collision>
     </link>
     <joint name="joint6" type="continuous">
@@ -104,4 +140,10 @@
             <material name="grey"/>
         </visual>
+        <collision>
+            <geometry>
+                <box size="0.15 0.1 0.02"/>
+            </geometry>
+            <origin xyz="0 0 0.01" rpy="0 0 0"/>
+        </collision>
     </link>
     <joint name="hand_tool_joint" type="fixed">
