Commit message: Fix: Uploading correct workspace files

File: src/kxsmoveit_robot_description/urdf/common_properties.xacro (robot description, xacro)
@@ -7,3 +7,9 @@
         <color rgba="0.0 0.0 1.0 1.0"/>
     </material>
+    <material name="dark_green">
+        <color rgba="0.0 0.4 0.0 1.0"/>
+    </material>
+    <material name="light_green">
+        <color rgba="0.0 0.6 0.0 1.0"/>
+    </material>
 </robot>

File: src/kxsmoveit_robot_description/urdf/kxsmoveit_robot.urdf.xacro (robot description, xacro)
@@ -3,3 +3,9 @@
     <xacro:include filename="common_properties.xacro"/>
     <xacro:include filename="arm.xacro"/>
+    <xacro:include filename="gripper.xacro"/>
+    <joint name="gripper_base_joint" type="fixed">
+        <parent link="tool_link"/>
+        <child link="gripper_base_link"/>
+        <origin xyz="0 0 0.0" rpy="0 0 0"/>
+    </joint>
 </robot>
